Commit message: 1122

File: config/ur5.urdf (robot description, URDF)
Before this commit: robot ur5, 12 links, 11 joints
Links:
- link ee_link: mass 0.001 -> 0.01
Joints:
- joint ee_joint: origin xyz=-0.03 0.085 0.03 rpy=-1.5707963267948966 0.0 0.0 -> xyz=0.03 0.085 -0.03 rpy=-1.5707963267948966 3.141592653589793238 0.0

File: config/ur5_endeffector_off.urdf (robot description, URDF)
Before this commit: robot ur5, 12 links, 11 joints
Links:
- link base_link: mass 4.0 -> 0.01
- link forearm_link: mass 2.2 -> 0.01
- link shoulder_link: mass 3.7 -> 0.01
- link upper_arm_link: mass 8.4 -> 0.01
- link wrist_1_link: mass 1.2 -> 0.01
- link wrist_2_link: mass 1.2 -> 0.01

Commit message: 1127

File: config/ur5.urdf (robot description, URDF)
Before this commit: robot ur5, 12 links, 11 joints
Links:
- link ee_link: mass 0.01 -> 0.1

Commit message: 12/12

File: config/ur5.urdf (robot description, URDF)
Before this commit: robot ur5, 12 links, 11 joints
Links:
- link tcp: mass None -> 0.000000001
